Commit message: Updated urdf file

File: quadruped/urdf/leg.urdf (robot description, URDF)
Before this commit: robot one_leg, 4 links, 3 joints
Links:
- removed link mild_link
- link link1: geometry collision mesh filename=../meshes/link1.STL scale=0.001 0.001 0.001; visual mesh filename=../meshes/link1.STL scale=0.001 0.001 0.001
- link link2: geometry collision mesh filename=../meshes/link2.STL scale=0.001 0.001 0.001; visual mesh filename=../meshes/link2.STL scale=0.001 0.001 0.001
Joints:
- removed joint mild_to_link1
- removed joint mild_to_rectangle
- added joint rectangle_to_link1: type revolute, parent rectangle, child link1, origin xyz=0.03 0.03 0.08 rpy=0 0 0, axis 0 0 1, limit lower=-1.57 upper=1.57 effort=100 velocity=10
- joint link1_to_link2: origin xyz=0.09272 0.07750 -0.00021 rpy=0 0 0 -> xyz=0.00041797 -0.12084033 0.00162 rpy=0 0 0
